Commit message: 5 Tasks - Laboratory 1

File: urdf/planar2dof.urdf (robot description, URDF)
Before this commit: robot planar2dof, 5 links, 4 joints
Links:
- link planar2dof/link_striker_ee: mass 0.1 -> 0.8

Commit message: lab2 done and lab1 fixed

File: urdf/planar2dof.urdf (robot description, URDF)
Before this commit: robot planar2dof, 5 links, 4 joints
Links:
- link planar2dof/link_striker_ee: mass 0.8 -> 0.1
